File: filterbuffer.kicad_pcb (KiCad board)
At the start: 2 copper layers, 143 x 45 mm, 27 parts, among them J1 Conn_01x02, J10 Conn_01x02, J11 Conn_01x02, J12 Conn_01x02, J13 Conn_01x02, J14 Conn_01x02, J15 Conn_01x02, J16 Conn_01x02, J2 Conn_01x02, J3 Conn_01x02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

Commit message: add system ground
Parts:
- H3: value MountingHole -> MountingHole_Pad; footprint MountingHole:MountingHole_3.2mm_M3 -> MountingHole:MountingHole_3.2mm_M3_Pad_Via
Connections:
- H3 pad 1: (no net) -> Net-(H3-Pad1)
Changed lines of the file:
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@@
     (zones 0)
     (modules 27)
-    (nets 10)
+    (nets 11)
   )
   (page A4)
@@
     (35 F.Paste user)
     (36 B.SilkS user)
-    (37 F.SilkS user hide)
+    (37 F.SilkS user)
     (38 B.Mask user)
     (39 F.Mask user)
@@
     (47 F.CrtYd user)
     (48 B.Fab user)
-    (49 F.Fab user hide)
+    (49 F.Fab user)
   )
   (setup
@@
     (pad_to_mask_clearance 0.051)
     (solder_mask_min_width 0.25)
-    (aux_axis_origin 0 0)
-    (grid_origin 121.45 151.45)
+    (aux_axis_origin 181.45 114.2)
+    (grid_origin 105.95 123.2)
     (visible_elements FFFFF77F)
     (pcbplotparams
@@
   (net 8 "Net-(D1-Pad2)")
   (net 9 "Net-(R2-Pad1)")
+  (net 10 "Net-(H3-Pad1)")
   (net_class Default "This is the default net class."
     (clearance 0.2)
@@
     (add_net "Net-(F1-Pad1)")
     (add_net "Net-(F1-Pad2)")
+    (add_net "Net-(H3-Pad1)")
     (add_net "Net-(R1-Pad1)")
     (add_net "Net-(R2-Pad1)")
     (add_net VCC)
+  )
+  (module MountingHole:MountingHole_3.2mm_M3_Pad_Via (layer F.Cu)
+    (at 181.45 114.2)
+    (descr "Mounting Hole 3.2mm, M3")
+    (tags "mounting hole 3.2mm m3")
+    (attr virtual)
+    (fp_text reference H3 (at 0 -4.2) (layer F.SilkS)
+      (effects (font (size 1 1) (thickness 0.15)))
+    )
+    (fp_text value MountingHole_Pad (at 0 4.2) (layer F.Fab)
+      (effects (font (size 1 1) (thickness 0.15)))
+    )
+    (fp_text user %R (at 0.3 0) (layer F.Fab)
+      (effects (font (size 1 1) (thickness 0.15)))
+    )
+    (fp_circle (center 0 0) (end 3.2 0) (layer Cmts.User) (width 0.15))
+    (fp_circle (center 0 0) (end 3.45 0) (layer F.CrtYd) (width 0.05))
+    (pad 1 thru_hole circle (at 0 0) (size 6.4 6.4) (drill 3.2) (layers *.Cu *.Mask)
+      (net 10 "Net-(H3-Pad1)"))
+    (pad 1 thru_hole circle (at 2.4 0) (size 0.8 0.8) (drill 0.5) (layers *.Cu *.Mask)
+      (net 10 "Net-(H3-Pad1)"))
+    (pad 1 thru_hole circle (at 1.697056 1.697056) (size 0.8 0.8) (drill 0.5) (layers *.Cu *.Mask)
+      (net 10 "Net-(H3-Pad1)"))
+    (pad 1 thru_hole circle (at 0 2.4) (size 0.8 0.8) (drill 0.5) (layers *.Cu *.Mask)
+      (net 10 "Net-(H3-Pad1)"))
+    (pad 1 thru_hole circle (at -1.697056 1.697056) (size 0.8 0.8) (drill 0.5) (layers *.Cu *.Mask)
+      (net 10 "Net-(H3-Pad1)"))
+    (pad 1 thru_hole circle (at -2.4 0) (size 0.8 0.8) (drill 0.5) (layers *.Cu *.Mask)
+      (net 10 "Net-(H3-Pad1)"))
+    (pad 1 thru_hole circle (at -1.697056 -1.697056) (size 0.8 0.8) (drill 0.5) (layers *.Cu *.Mask)
+      (net 10 "Net-(H3-Pad1)"))
+    (pad 1 thru_hole circle (at 0 -2.4) (size 0.8 0.8) (drill 0.5) (layers *.Cu *.Mask)
+      (net 10 "Net-(H3-Pad1)"))
+    (pad 1 thru_hole circle (at 1.697056 -1.697056) (size 0.8 0.8) (drill 0.5) (layers *.Cu *.Mask)
+      (net 10 "Net-(H3-Pad1)"))
   )
   (module MountingHole:MountingHole_3.2mm_M3 (layer F.Cu)
@@
     (pad 1 np_thru_hole circle (at 0 0) (size 3.2 3.2) (drill 3.2) (layers *.Cu *.Mask))
   )
-  (module MountingHole:MountingHole_3.2mm_M3 (layer F.Cu)
-    (at 181.45 114.2)
-    (descr "Mounting Hole 3.2mm, no annular, M3")
-    (tags "mounting hole 3.2mm no annular m3")
-    (attr virtual)
-    (fp_text reference H3 (at 0 -4.2) (layer F.SilkS)
-      (effects (font (size 1 1) (thickness 0.15)))
-    )
-    (fp_text value MountingHole (at 0 4.2) (layer F.Fab)
-      (effects (font (size 1 1) (thickness 0.15)))
-    )
-    (fp_text user %R (at 0.3 0) (layer F.Fab)
-      (effects (font (size 1 1) (thickness 0.15)))
-    )
-    (fp_circle (center 0 0) (end 3.2 0) (layer Cmts.User) (width 0.15))
-    (fp_circle (center 0 0) (end 3.45 0) (layer F.CrtYd) (width 0.05))
-    (pad 1 np_thru_hole circle (at 0 0) (size 3.2 3.2) (drill 3.2) (layers *.Cu *.Mask))
-  )

Commit message: layout redesign
Parts:
- J10, J12, J13, J15, J3, J4, J6, J7, J9: footprint Sockets_MOLEX_KK-System:Socket_MOLEX-KK-RM2-54mm_Lock_2pin_straight -> Connector_PinHeader_2.54mm:PinHeader_1x02_P2.54mm_Vertical
- moved R1 26.0 mm to (74.7, 129.9)
- moved R2 26.0 mm to (78.0, 129.9)
- moved R3 26.0 mm to (81.2, 129.9)
- moved D1 25.9 mm to (76.1, 134.4)
- moved TH1 15.0 mm to (169.7, 119.0), turned to 90 degrees
- moved J10 12.6 mm to (62.2, 106.0)
- moved H2 12.5 mm to (62.0, 115.5)
- moved J11 12.2 mm to (68.4, 131.2)
- moved J7 11.6 mm to (67.7, 106.0)
- moved J16 11.4 mm to (170.2, 129.0), turned to 90 degrees
- moved J5 10.7 mm to (61.7, 131.2)
- moved J4 10.5 mm to (73.2, 106.0)
- moved H3 10.0 mm to (180.7, 104.2)
- moved J1 9.77 mm to (61.7, 123.7)
- moved F1 9.72 mm to (180.2, 133.7)
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Routing:
- net Net-(D1-Pad2): track 3.52 -> 3.02 mm
Other:
- board size 143 x 45 mm -> 128.5 x 38 mm
