File: filterbuffer.sch (KiCad schematic (older format))
At the start: 27 parts, among them J1 Conn_01x02, J10 Conn_01x02, J11 Conn_01x02, J12 Conn_01x02, J13 Conn_01x02, J14 Conn_01x02, J15 Conn_01x02, J16 Conn_01x02, J2 Conn_01x02, J3 Conn_01x02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

Commit message: add system ground
Parts:
- removed H3: MountingHole, MountingHole:MountingHole_3.2mm_M3, symbol Mechanical:MountingHole
- added H3: MountingHole_Pad, MountingHole:MountingHole_3.2mm_M3_Pad_Via, symbol Mechanical:MountingHole_Pad
Changed lines of the file:
@@
-$EndComp
-$Comp
-L Mechanical:MountingHole H3
-U 1 1 5CB1D52B
-P 1600 2950
-F 0 "H3" H 1700 2996 50  0000 L CNN
-F 1 "MountingHole" H 1700 2905 50  0000 L CNN
-F 2 "MountingHole:MountingHole_3.2mm_M3" H 1600 2950 50  0001 C CNN
-F 3 "~" H 1600 2950 50  0001 C CNN
-	1    1600 2950
-	1    0    0    -1
 $EndComp
 $Comp
@@
 	1    0    0    -1
 $EndComp
+$Comp
+L Mechanical:MountingHole_Pad H3
+U 1 1 5CB27581
+P 1600 3000
+F 0 "H3" H 1700 3051 50  0000 L CNN
+F 1 "MountingHole_Pad" H 1700 2960 50  0000 L CNN
+F 2 "MountingHole:MountingHole_3.2mm_M3_Pad_Via" H 1600 3000 50  0001 C CNN
+F 3 "~" H 1600 3000 50  0001 C CNN
+	1    1600 3000
+	1    0    0    -1
+$EndComp

Commit message: layout redesign
Parts:
- J10, J12, J13, J15, J3, J4, J6, J7, J9: footprint Sockets_MOLEX_KK-System:Socket_MOLEX-KK-RM2-54mm_Lock_2pin_straight -> Connector_PinHeader_2.54mm:PinHeader_1x02_P2.54mm_Vertical
Changed lines of the file:
@@
 F 0 "J10" V 4166 1012 50  0000 R CNN
 F 1 "Conn_01x02" V 4075 1012 50  0000 R CNN
-F 2 "Sockets_MOLEX_KK-System:Socket_MOLEX-KK-RM2-54mm_Lock_2pin_straight" H 4200 1200 50  0001 C CNN
+F 2 "Connector_PinHeader_2.54mm:PinHeader_1x02_P2.54mm_Vertical" H 4200 1200 50  0001 C CNN
 F 3 "~" H 4200 1200 50  0001 C CNN
 	1    4200 1200
@@
 F 0 "J13" V 4466 1012 50  0000 R CNN
 F 1 "Conn_01x02" V 4375 1012 50  0000 R CNN
-F 2 "Sockets_MOLEX_KK-System:Socket_MOLEX-KK-RM2-54mm_Lock_2pin_straight" H 4500 1200 50  0001 C CNN
+F 2 "Connector_PinHeader_2.54mm:PinHeader_1x02_P2.54mm_Vertical" H 4500 1200 50  0001 C CNN
 F 3 "~" H 4500 1200 50  0001 C CNN
 	1    4500 1200
@@
 F 0 "J7" V 3866 1012 50  0000 R CNN
 F 1 "Conn_01x02" V 3775 1012 50  0000 R CNN
-F 2 "Sockets_MOLEX_KK-System:Socket_MOLEX-KK-RM2-54mm_Lock_2pin_straight" H 3900 1200 50  0001 C CNN
+F 2 "Connector_PinHeader_2.54mm:PinHeader_1x02_P2.54mm_Vertical" H 3900 1200 50  0001 C CNN
 F 3 "~" H 3900 1200 50  0001 C CNN
 	1    3900 1200
@@
 F 0 "J4" V 3566 1012 50  0000 R CNN
 F 1 "Conn_01x02" V 3475 1012 50  0000 R CNN
-F 2 "Sockets_MOLEX_KK-System:Socket_MOLEX-KK-RM2-54mm_Lock_2pin_straight" H 3600 1200 50  0001 C CNN
+F 2 "Connector_PinHeader_2.54mm:PinHeader_1x02_P2.54mm_Vertical" H 3600 1200 50  0001 C CNN
 F 3 "~" H 3600 1200 50  0001 C CNN
 	1    3600 1200
@@
 F 0 "J15" V 4916 1012 50  0000 R CNN
 F 1 "Conn_01x02" V 4825 1012 50  0000 R CNN
-F 2 "Sockets_MOLEX_KK-System:Socket_MOLEX-KK-RM2-54mm_Lock_2pin_straight" H 4950 1200 50  0001 C CNN
+F 2 "Connector_PinHeader_2.54mm:PinHeader_1x02_P2.54mm_Vertical" H 4950 1200 50  0001 C CNN
 F 3 "~" H 4950 1200 50  0001 C CNN
 	1    4950 1200
@@
 F 0 "J3" V 3373 3280 50  0000 L CNN
 F 1 "Conn_01x02" V 3464 3280 50  0000 L CNN
-F 2 "Sockets_MOLEX_KK-System:Socket_MOLEX-KK-RM2-54mm_Lock_2pin_straight" H 3500 3200 50  0001 C CNN
+F 2 "Connector_PinHeader_2.54mm:PinHeader_1x02_P2.54mm_Vertical" H 3500 3200 50  0001 C CNN
 F 3 "~" H 3500 3200 50  0001 C CNN
 	1    3500 3200
@@
 F 0 "J6" V 3673 3280 50  0000 L CNN
 F 1 "Conn_01x02" V 3764 3280 50  0000 L CNN
-F 2 "Sockets_MOLEX_KK-System:Socket_MOLEX-KK-RM2-54mm_Lock_2pin_straight" H 3800 3200 50  0001 C CNN
+F 2 "Connector_PinHeader_2.54mm:PinHeader_1x02_P2.54mm_Vertical" H 3800 3200 50  0001 C CNN
 F 3 "~" H 3800 3200 50  0001 C CNN
 	1    3800 3200
@@
 F 0 "J9" V 3973 3280 50  0000 L CNN
 F 1 "Conn_01x02" V 4064 3280 50  0000 L CNN
-F 2 "Sockets_MOLEX_KK-System:Socket_MOLEX-KK-RM2-54mm_Lock_2pin_straight" H 4100 3200 50  0001 C CNN
+F 2 "Connector_PinHeader_2.54mm:PinHeader_1x02_P2.54mm_Vertical" H 4100 3200 50  0001 C CNN
 F 3 "~" H 4100 3200 50  0001 C CNN
 	1    4100 3200
@@
 F 0 "J12" V 4273 3280 50  0000 L CNN
 F 1 "Conn_01x02" V 4364 3280 50  0000 L CNN
-F 2 "Sockets_MOLEX_KK-System:Socket_MOLEX-KK-RM2-54mm_Lock_2pin_straight" H 4400 3200 50  0001 C CNN
+F 2 "Connector_PinHeader_2.54mm:PinHeader_1x02_P2.54mm_Vertical" H 4400 3200 50  0001 C CNN
 F 3 "~" H 4400 3200 50  0001 C CNN
 	1    4400 3200

Commit message: update layout
Parts:
- removed J4: Conn_01x02, Connector_PinHeader_2.54mm:PinHeader_1x02_P2.54mm_Vertical, symbol Connector_Generic:Conn_01x02
- added H4: MountingHole, MountingHole:MountingHole_3.2mm_M3, symbol Mechanical:MountingHole
- added J18: Conn_01x02, Connector_PinHeader_2.54mm:PinHeader_1x02_P2.54mm_Vertical, symbol Connector_Generic:Conn_01x02
- F1: footprint Fuse:Fuseholder_Cylinder-5x20mm_Stelvio-Kontek_PTF78_Horizontal_Open -> 696105003002:FUSE_696105003002
- J1, J11, J14, J16, J5, J8: footprint Sockets_MOLEX_KK-System:Socket_MOLEX-KK-RM2-54mm_Lock_2pin_straight -> TerminalBlock_Phoenix:TerminalBlock_Phoenix_PT-1,5-2-3.5-H_1x02_P3.50mm_Horizontal
- J2: footprint Sockets_MOLEX_KK-System:Socket_MOLEX-KK-RM2-54mm_Lock_2pin_straight -> Connector_PinHeader_2.54mm:PinHeader_1x02_P2.54mm_Vertical
Connections:
- net +12V: now also J18.2 (Pin_2)
- net +5V: now also J2.1 (Pin_1)
- net GND: now also H3.1, J18.1 (Pin_1)
- net VCC: no longer J2.1 (Pin_1)
Other:
- moved on the sheet: J15
